Commit message: Get real robot working.

File: diffbot_description/urdf/diffbot.ros2_control.xacro (robot description, xacro)
@@ -2,5 +2,31 @@
 <robot xmlns:xacro="http://www.ros.org/wiki/xacro">
     <xacro:macro name="diffbot_ros2_control">
-        <ros2_control name="diffbot_hardware_interface" type="system">
+        <ros2_control name="RealRobot" type="system">
+            <hardware>
+                <plugin>diffdrive_arduino/DiffDriveArduino</plugin>
+                <param name="left_wheel_name">left_wheel_joint</param>
+                <param name="right_wheel_name">right_wheel_joint</param>
+                <param name="loop_rate">30</param>
+                <param name="device">/dev/ttyUSB0</param>
+                <param name="baud_rate">57600</param>
+                <param name="timeout">1000</param>
+                <param name="enc_counts_per_rev">3450</param>
+            </hardware>
+            <joint name="left_wheel_joint">
+                <command_interface name="velocity"/>
+                    <param name="min">-10</param>
+                    <param name="max">10</param>
+                <state_interface name="position"/>
+                <state_interface name="velocity"/>
+            </joint>
+            <joint name="right_wheel_joint">
+                <command_interface name="velocity"/>
+                    <param name="min">-10</param>
+                    <param name="max">10</param>
+                <state_interface name="position"/>
+                <state_interface name="velocity"/>
+            </joint>
+        </ros2_control>
+        <!--<ros2_control name="diffbot_hardware_interface" type="system">
             <hardware>
                 <plugin>gz_ros2_control/GazeboSimSystem</plugin>
@@ -20,5 +46,5 @@
                 <state_interface name="velocity"/>
             </joint>
-        </ros2_control>
+        </ros2_control>-->
     </xacro:macro>
     <gazebo>

Commit message: ros2 control

File: diffbot_description/urdf/diffbot.ros2_control.xacro (robot description, xacro)
@@ -2,5 +2,5 @@
 <robot xmlns:xacro="http://www.ros.org/wiki/xacro">
     <xacro:macro name="diffbot_ros2_control">
-        <ros2_control name="RealRobot" type="system">
+        <!--<ros2_control name="RealRobot" type="system">
             <hardware>
                 <plugin>diffdrive_arduino/DiffDriveArduino</plugin>
@@ -27,6 +27,6 @@
                 <state_interface name="velocity"/>
             </joint>
-        </ros2_control>
-        <!--<ros2_control name="diffbot_hardware_interface" type="system">
+        </ros2_control>-->
+        <ros2_control name="diffbot_hardware_interface" type="system">
             <hardware>
                 <plugin>gz_ros2_control/GazeboSimSystem</plugin>
@@ -46,5 +46,5 @@
                 <state_interface name="velocity"/>
             </joint>
-        </ros2_control>-->
+        </ros2_control>
     </xacro:macro>
     <gazebo>

File: diffbot_description/urdf/diffbot.urdf.xacro (robot description, xacro)
@@ -2,4 +2,5 @@
 <robot xmlns:xacro="http://www.ros.org/wiki/xacro"  name="diffbot_robot">
   <xacro:include filename="diffbot_description.urdf.xacro"/>
+  <xacro:include filename="lidar.xacro"/>
   <xacro:include filename="diffbot.ros2_control.xacro"/>
   <xacro:diffbot_ros2_control/>

File: diffbot_description/urdf/diffbot_description.urdf.xacro (robot description, xacro)
@@ -18,9 +18,9 @@
     <parent link="base_footprint"/>
     <child link="base_link"/>
-    <origin xyz="0 0 0.05"/>
+    <origin xyz="0.3 0 0.05"/>
   </joint>
   <link name="base_link">
     <visual>
-      <origin xyz="0.15 0 0.075"/>
+      <origin xyz="-0.15 0 0.075"/>
       <geometry>
         <box size="0.3 0.3 0.15"/>
@@ -29,5 +29,5 @@
     </visual>
     <collision>
-      <origin xyz="0.15 0 0.075"/>
+      <origin xyz="-0.15 0 0.075"/>
       <geometry>
         <box size="0.3 0.3 0.15"/>
@@ -35,5 +35,5 @@
     </collision>
     <xacro:inertial_box mass="0.5" x="0.3" y="0.3" z="0.15">
-      <origin xyz="0.15 0 0.075" rpy="0 0 0"/>
+      <origin xyz="-0.15 0 0.075" rpy="0 0 0"/>
     </xacro:inertial_box>
   </link>
@@ -42,8 +42,31 @@
     <parent link="base_link"/>
     <child link="left_wheel"/>
-    <origin xyz="0.05 0.175 0" rpy="-${pi/2} 0 0"/>
+    <origin xyz="0 0.175 0" rpy="-${pi/2} 0 0"/>
     <axis xyz="0 0 1"/>
   </joint>
   <link name="left_wheel">
+    <visual>
+      <geometry>
+        <cylinder radius="0.05" length="0.04"/>
+      </geometry>
+      <material name="blue"/>
+    </visual>
+    <collision>
+      <geometry>
+        <cylinder radius="0.05" length="0.04"/>
+      </geometry>
+    </collision>
+    <xacro:inertial_cylinder mass="0.1" length="0.04" radius="0.05">
+      <origin xyz="0 0 0" rpy="0 0 0"/>
+    </xacro:inertial_cylinder>
+  </link>
+  <!-- left_dummy -->
+  <joint name="left_dummy_joint" type="continuous">
+    <parent link="base_link"/>
+    <child link="left_dummy"/>
+    <origin xyz="-0.3 0.175 0" rpy="-${pi/2} 0 0"/>
+    <axis xyz="0 0 1"/>
+  </joint>
+  <link name="left_dummy">
     <visual>
       <geometry>
@@ -65,5 +88,5 @@
     <parent link="base_link"/>
     <child link="right_wheel"/>
-    <origin xyz="0.05 -0.175 0" rpy="${pi/2} 0 0"/>
+    <origin xyz="0 -0.175 0" rpy="${pi/2} 0 0"/>
     <axis xyz="0 0 -1"/>
   </joint>
@@ -84,5 +107,28 @@
     </xacro:inertial_cylinder>
   </link>
-  <!-- caster frontal wheel Link -->
+  <!-- right_dummy -->
+  <joint name="right_dummy_joint" type="continuous">
+    <parent link="base_link"/>
+    <child link="right_dummy"/>
+    <origin xyz="-0.3 -0.175 0" rpy="${pi/2} 0 0"/>
+    <axis xyz="0 0 -1"/>
+  </joint>
+  <link name="right_dummy">
+    <visual>
+      <geometry>
+        <cylinder radius="0.05" length="0.04"/>
+      </geometry>
+      <material name="blue"/>
+    </visual>
+    <collision>
+      <geometry>
+        <cylinder radius="0.05" length="0.04"/>
+      </geometry>
+    </collision>
+    <xacro:inertial_cylinder mass="0.1" length="0.04" radius="0.05">
+      <origin xyz="0 0 0" rpy="0 0 0"/>
+    </xacro:inertial_cylinder>
+  </link>
+  <!-- caster frontal wheel Link
   <joint name="caster_wheel_joint" type="fixed">
     <parent link="base_link"/>
@@ -105,9 +151,9 @@
       <origin xyz="0 0 0" rpy="0 0 0"/>
     </xacro:inertial_sphere>
-  </link>
-  <gazebo reference="caster_wheel">
-    <!-- <material>Gazebo/orange</material> -->
+  </link>-->
+  <!--<gazebo reference="caster_wheel">
+     <material>Gazebo/orange</material>
     <mu1 value="0.001"/>
     <mu2 value="0.001"/>
-  </gazebo>
+  </gazebo>-->
 </robot>
